File: senior_design.kicad_sch (KiCad schematic)
At the start: 12 parts, among them U1 STM32L152RETx, U2 AHT20, U3 BMP280

Commit message: Add files via upload
Parts:
- removed U2: AHT20, AHT20:PSON100P300X300X110-6N, symbol AHT20:AHT20
- removed U3: BMP280, Package_LGA:Bosch_LGA-8_2x2.5mm_P0.65mm_ClockwisePinNumbering, symbol Sensor_Pressure:BMP280
- added C10, C9: C, symbol Device:C
- added J1: Conn_01x04_Pin, symbol Connector:Conn_01x04_Pin
- added Y1: Crystal_GND24, symbol Device:Crystal_GND24
- C5: value 10u -> 4.7u
Connections:
- net +3.3V: now also J1.4 (Pin_4)
- net +3.3VA: now also U1.13 (VDDA)
- net GND: now also C10.2, C9.2, J1.1 (Pin_1), Y1.2 (G), Y1.4 (G)
- new net: C10.1, Y1.3
- new net: C9.1, Y1.1
Other:
- note added: "HSE_IN"
- note added: "HSE_out"
- note added: "Here's the crystal, we need to attach it to HSE_in and HSE_out"
- note added: "I2C1_SCL"
- note added: "I2C1_SDA"
- note added: "RCC_OSC32_IN"
- note added: "RCC_OSC32_OUT"
- note added: "RCC_OSC_IN"
- note added: "RCC_OSC_OUT"
- note added: "TCK"
- note added: "TMS"
- note added: "USART1_RX"
- note added: "USART1_TX"
- note added: "USART_RX"
- note added: "USART_TX"
- note added: "blue_pushbutton"
- note added: "green_led"
- note added: "here's the debugger, we need to connect swdio and swclk to the corresponding pins"
- note added: "swclk"
- note added: "swdio"
